Commit message: 6轴绝对值编码器闭环版本
增加初始姿态识别功能，可由传感器获取机器人关节数据，同时此API为机器人提供示教功能实现的基础

File: tgr_arm_description/urdf/tgr_arm.urdf (robot description, URDF)
Before this commit: robot tgr_arm, 7 links, 6 joints
Joints:
- joint joint3: axis 1 0 0 -> 0 0 1; origin xyz=0.085 0 0 rpy=0 0 0 -> xyz=0 0 0.085 rpy=0 0 0
- joint joint4: origin xyz=0.145 0 0 rpy=0 0 0 -> xyz=0 0 0.145 rpy=0 0 0
- joint joint5: origin xyz=0 -0.00018 -0.068 rpy=0 3.1415926 0 -> xyz=0 0 0.11 rpy=0 0 0
